File: RiftBoard.kicad_sch (KiCad schematic)
At the start: 38 parts, among them J1 USB_C_Receptacle_USB2.0_14P, J2 Conn_01x20, J3 Conn_01x20, J4 Conn_01x03, SW1 SW_Push, SW2 SW_Push, U1 RP2040, U2 MCP1700x-330xxTT, U3 W25Q16JVUXIQ TR, Y1 12MHz

Commit message: Finished PCB stuffs, now just design and I can move on to the production and assembly.
Connections:
- net GPIO17: now also SW2.1; no longer J3.6 (Pin_6)
- net GPIO18: now also J3.17 (Pin_17); no longer J3.7 (Pin_7)
- net GPIO19: now also J3.15 (Pin_15); no longer J3.8 (Pin_8)
- net GPIO20: now also J3.14 (Pin_14); no longer J3.9 (Pin_9)
- net GPIO21: now also J3.13 (Pin_13); no longer J3.10 (Pin_10)
- net GPIO22: now also J3.12 (Pin_12); no longer J3.17 (Pin_17)
- net GPIO23: now also J3.10 (Pin_10); no longer SW2.1
- net GPIO26/ADC0: now also J3.7 (Pin_7); no longer J3.12 (Pin_12)
- net GPIO27/ADC1: now also J3.6 (Pin_6); no longer J3.13 (Pin_13)
- net GPIO28/ADC2: now also J3.5 (Pin_5); no longer J3.14 (Pin_14)
- net GPIO29/ADC3: now also J3.4 (Pin_4); no longer J3.15 (Pin_15)
- net at R8.1: now also U1.18 (GPIO15); no longer U1.36 (GPIO24)
- net at R9.1: now also U1.27 (GPIO16); no longer U1.37 (GPIO25)
- removed net GPIO15: J3.4 (Pin_4), U1.18 (GPIO15)
- removed net GPIO16: J3.5 (Pin_5), U1.27 (GPIO16)
- new net GPIO24: J3.9 (Pin_9), U1.36 (GPIO24)
- new net GPIO25: J3.8 (Pin_8), U1.37 (GPIO25)
Other:
- moved on the sheet: D1, D2, R8, R9

Commit message: submission
Parts:
- removed J1: USB_C_Receptacle_USB2.0_14P, Connector_USB:USB_C_Receptacle_HRO_TYPE-C-31-M-12, symbol Connector:USB_C_Receptacle_USB2.0_14P
- added J1: USB_C_Receptacle_USB2.0_16P, Connector_USB:USB_C_Receptacle_HRO_TYPE-C-31-M-12, symbol Connector:USB_C_Receptacle_USB2.0_16P
Connections:
- net GND: now also J1.A1 (GND), J1.A12 (GND), J1.B1 (GND), J1.B12 (GND), J1.S1 (SHIELD)
- net USB_D+: now also J1.A6 (D+), J1.B6 (D+)
- net USB_D-: now also J1.A7 (D-), J1.B7 (D-)
- net VBUS: now also J1.A4 (VBUS), J1.A9 (VBUS), J1.B4 (VBUS), J1.B9 (VBUS)
- net at R1.1: now also J1.A5 (CC1)
- net at R2.1: now also J1.B5 (CC2)
- no-connect marks 0 -> 2
Changed lines of the file:
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@@
 		(color 0 0 0 0)
 	)
+	(no_connect
+		(at 45.72 62.23)
+	)
+	(no_connect
+		(at 45.72 59.69)
+	)
 	(wire
 		(pts
@@
 	)
 	(symbol
-		(lib_id "Connector:USB_C_Receptacle_USB2.0_14P")
-		(at 30.48 46.99 0)
-		(unit 1)
-		(exclude_from_sim no)
-		(in_bom yes)
-		(on_board yes)
-		(dnp no)
-		(fields_autoplaced yes)
-		(property "Reference" "J1"
-			(at 30.48 24.13 0)
-			(effects
-				(font
-					(size 1.27 1.27)
-				)
-			)
-		)
-		(property "Value" "USB_C_Receptacle_USB2.0_14P"
-			(at 30.48 26.67 0)
-			(effects
-				(font
-					(size 1.27 1.27)
-				)
-			)
-		)
-		(property "Footprint" "Connector_USB:USB_C_Receptacle_HRO_TYPE-C-31-M-12"
-			(at 34.29 46.99 0)
-			(effects
-				(font
-					(size 1.27 1.27)
-				)
-				(hide yes)
-			)
-		)
-		(property "Datasheet" "https://www.usb.org/sites/default/files/documents/usb_type-c.zip"
-			(at 34.29 46.99 0)
-			(effects
-				(font
-					(size 1.27 1.27)
-				)
-				(hide yes)
-			)
-		)
-		(property "Description" "USB 2.0-only 14P Type-C Receptacle connector"
-			(at 30.48 46.99 0)
-			(effects
-				(font
-					(size 1.27 1.27)
-				)
-				(hide yes)
-			)
-		)
-		(pin "B5"
-		)
-		(pin "A6"
-		)
-		(pin "A7"
-		)
-		(pin "B7"
-		)
-		(pin "B6"
-		)
-		(pin "A9"
-		)
-		(pin "B4"
-		)
-		(pin "B9"
-		)
-		(pin "A5"
-		)
-		(pin "A1"
-		)
-		(pin "A12"
-		)
-		(pin "S1"
-		)
-		(pin "B1"
-		)
-		(pin "A4"
-		)
-		(pin "B12"
-		)
-		(instances
-			(project ""
-				(path "/f03da10f-a927-4e36-a5be-925c35c78d2a"
-					(reference "J1")
-					(unit 1)
-				)
-			)
-		)
-	)
-	(symbol
 		(lib_id "power:GND")
 		(at 20.32 114.3 0)
@@
 	)
 	(symbol
+		(lib_id "Connector:USB_C_Receptacle_USB2.0_16P")
+		(at 30.48 46.99 0)
+		(unit 1)
+		(exclude_from_sim no)
+		(in_bom yes)
+		(on_board yes)
+		(dnp no)
+		(fields_autoplaced yes)
+		(property "Reference" "J1"
+			(at 30.48 24.13 0)
+			(effects
+				(font
+					(size 1.27 1.27)
+				)
+			)
+		)
+		(property "Value" "USB_C_Receptacle_USB2.0_16P"
+			(at 30.48 26.67 0)
+			(effects
+				(font
+					(size 1.27 1.27)
+				)
+			)
+		)
+		(property "Footprint" "Connector_USB:USB_C_Receptacle_HRO_TYPE-C-31-M-12"
+			(at 34.29 46.99 0)
+			(effects
+				(font
+					(size 1.27 1.27)
+				)
+				(hide yes)
+			)
+		)
+		(property "Datasheet" "https://www.usb.org/sites/default/files/documents/usb_type-c.zip"
+			(at 34.29 46.99 0)
+			(effects
+				(font
+					(size 1.27 1.27)
+				)
+				(hide yes)
+			)
+		)
+		(property "Description" "USB 2.0-only 16P Type-C Receptacle connector"
+			(at 30.48 46.99 0)
+			(effects
+				(font
+					(size 1.27 1.27)
+				)
+				(hide yes)
+			)
+		)
+		(pin "B9"
+		)
+		(pin "B5"
+		)
+		(pin "A7"
+		)
+		(pin "B1"
+		)
+		(pin "A1"
+		)
+		(pin "B12"
+		)
+		(pin "S1"
+		)
+		(pin "A9"
+		)
+		(pin "B4"
+		)
+		(pin "A12"
+		)
+		(pin "A4"
+		)
+		(pin "A5"
+		)
+		(pin "A6"
+		)
+		(pin "B6"
+		)
+		(pin "A8"
+		)
+		(pin "B8"
+		)
+		(pin "B7"
+		)
+		(instances
+			(project ""
+				(path "/f03da10f-a927-4e36-a5be-925c35c78d2a"
+					(reference "J1")
+					(unit 1)
+				)
+			)
+		)
+	)
+	(symbol
 		(lib_id "power:GND")
 		(at 73.66 104.14 90)
@@
 		(dnp no)
 		(property "Reference" "D2"
-			(at 179.07 116.332 0)
+			(at 179.07 115.316 0)
 			(effects
 				(font
@@
 		)
 		(property "Value" "RED"
-			(at 179.832 111.506 0)
+			(at 182.372 111.76 0)
 			(effects
 				(font
@@
 		(dnp no)
 		(property "Reference" "D1"
-			(at 178.054 119.38 0)
+			(at 179.07 117.348 0)
 			(effects
 				(font
@@
 		)
 		(property "Value" "BLUE"
-			(at 178.054 117.856 0)
+			(at 182.626 119.126 0)
 			(effects
 				(font
